File: hardware/neogeo-diag-mvs-prog.kicad_pcb (KiCad board)
At the start: 2 copper layers, 174 x 134 mm, 21 parts, among them J1 NeoGeo MVS Prog B Side Edge, J2 NeoGeo MVS Prog A Side Edge, J3 NeoGeo MVS Prog B Side Edge, J4 NeoGeo MVS Prog A Side Edge, U1 AS6C8016, U2 74LS11, U3 74LS08, U4 74LS04

Commit message: Lower edge connector pads a little bit
Parts:
- moved J1 0.41 mm to (138.5, 150.7)
- moved J2 0.41 mm to (141.0, 150.7)
Other:
- board text added: "NEOGEO DIAG MVS PROG ${REV}"
- board text added: "PORTADRS (HALF)"
- board text added: "ROMOE (DIM)"
- board text added: "SLOTCS (FULL)"
- board text removed: "NEO-GEO DIAG MVS PROG ${REV}"
- board text removed: "NEO-GEO DIAG MVS PROG 2023-02-05"
Changed lines of the file:
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@@
   )
   (paper "A4")
+  (title_block
+    (title "NeoGeo Diag MVS Prog Board")
+    (date "${REV}")
+    (rev "${REV}")
+  )
   (layers
     (0 "F.Cu" signal)
@@
   (net 115 "unconnected-(U3-Pad13)")
   (footprint "neogeo-diag:neogeo-mvs-prog-a-side-edge" (layer "F.Cu")
-    (at 141 150.241)
+    (at 141 150.65)
     (property "Sheetfile" "neogeo-diag-mvs-prog.kicad_sch")
     (property "Sheetname" "")
@@
   )
   (footprint "neogeo-diag:neogeo-mvs-prog-b-side-edge" (layer "B.Cu")
-    (at 138.46 150.241 180)
+    (at 138.46 150.65 180)
     (property "Sheetfile" "neogeo-diag-mvs-prog.kicad_sch")
     (property "Sheetname" "")
@@
   (gr_circle (center 159.1818 103.759) (end 159.556827 103.759) (layer "F.SilkS") (width 0.15) (fill solid))
   (gr_circle (center 123.9266 112.776) (end 124.301627 112.776) (layer "F.SilkS") (width 0.15) (fill solid))
-  (gr_rect (start 216.75 145.234) (end 62.75 157.75) (layer "B.Mask") (width 0) (fill solid))
-  (gr_rect (start 62.75 145.234) (end 216.75 157.75) (layer "F.Mask") (width 0) (fill solid))
+  (gr_rect (start 216.95 145.65) (end 62.45 158.166) (layer "B.Mask") (width 0) (fill solid))
+  (gr_rect (start 62.5 145.65) (end 217 157.75) (layer "F.Mask") (width 0) (fill solid))
   (gr_line (start 100.75 26.25) (end 100.75 23.75) (layer "Edge.Cuts") (width 0.1))
   (gr_line (start 226.75 138.75) (end 226.75 23.75) (layer "Edge.Cuts") (width 0.1))
   (gr_line (start 100.75 23.75) (end 178.75 23.75) (layer "Edge.Cuts") (width 0.1))
-  (gr_line (start 217.05 157.75) (end 217.05 138.76) (layer "Edge.Cuts") (width 0.1))
+  (gr_line (start 217.05 157.75) (end 217.05 138.75) (layer "Edge.Cuts") (width 0.1))
   (gr_line (start 52.75 138.75) (end 52.75 23.75) (layer "Edge.Cuts") (width 0.1))
   (gr_circle (center 184.75 127) (end 189.75 127) (layer "Edge.Cuts") (width 0.1) (fill none))
@@
     (effects (font (size 0.7 0.7) (thickness 0.12)) (justify right mirror))
   )
-  (gr_text "NEO-GEO DIAG\nMVS PROG\n2023-02-05" (at 213 39.75) (layer "B.SilkS")
+  (gr_text "NEOGEO DIAG\nMVS PROG\n${REV}" (at 213 39.75) (layer "B.SilkS")
     (effects (font (size 1 1) (thickness 0.15)) (justify mirror))
   )
@@
     (effects (font (size 0.7 0.7) (thickness 0.12)) (justify right))
   )
-  (gr_text "NEO-GEO DIAG\nMVS PROG\n${REV}" (at 213 39.75) (layer "F.SilkS")
+  (gr_text "NEOGEO DIAG\nMVS PROG\n${REV}" (at 213 39.75) (layer "F.SilkS")
     (effects (font (size 1 1) (thickness 0.15)))
   )
@@
     (effects (font (size 0.7 0.7) (thickness 0.12)) (justify left))
   )
-  (gr_text "SLOTCS" (at 121.7168 94.3356 90) (layer "F.SilkS")
-    (effects (font (size 1 1) (thickness 0.15)))
+  (gr_text "SLOTCS (FULL)" (at 121.7168 97.282 90) (layer "F.SilkS")
+    (effects (font (size 1 1) (thickness 0.15)) (justify left))
   )
   (gr_text "NC38A" (at 120.65 140.716 90) (layer "F.SilkS")
@@
     (effects (font (size 0.7 0.7) (thickness 0.12)) (justify right))
   )
-  (gr_text "ROMOE" (at 133.858 94.5896 90) (layer "F.SilkS")
-    (effects (font (size 1 1) (thickness 0.15)))
+  (gr_text "ROMOE (DIM)" (at 133.858 97.282 90) (layer "F.SilkS")
+    (effects (font (size 1 1) (thickness 0.15)) (justify left))
   )
   (gr_text "A6" (at 191.77 136.144 90) (layer "F.SilkS")
@@
     (effects (font (size 0.7 0.7) (thickness 0.12)) (justify right))
   )
-  (gr_text "PORTADRS" (at 127.8128 93.3704 90) (layer "F.SilkS")
-    (effects (font (size 1 1) (thickness 0.15)))
+  (gr_text "PORTADRS (HALF)" (at 127.8128 97.282 90) (layer "F.SilkS")
+    (effects (font (size 1 1) (thickness 0.15)) (justify left))
   )
   (gr_text "D7" (at 186.69 140.716 90) (layer "F.SilkS")
@@
     (polygon
       (pts
-        (xy 73.17 155.24)
-        (xy 64.05 155.24)
+        (xy 73.17 155.65)
+        (xy 64.05 155.65)
         (xy 64.05 135)
         (xy 73.17 135)
@@
     (polygon
       (pts
-        (xy 215.41 155.24)
-        (xy 206.29 155.24)
+        (xy 215.41 155.65)
+        (xy 206.29 155.65)
         (xy 206.29 135)
         (xy 215.41 135)
@@
     (polygon
       (pts
-        (xy 144.292 145.239974)
-        (xy 144.292 155.239974)
-        (xy 135.172 155.239974)
-        (xy 135.172 145.239974)
+        (xy 144.29 145.65)
+        (xy 144.29 155.65)
+        (xy 135.17 155.65)
+        (xy 135.17 145.65)
         (xy 137.162 138.429974)
         (xy 142.242 138.429974)
@@
     (polygon
       (pts
-        (xy 215.409952 155.239998)
-        (xy 206.290035 155.24)
+        (xy 215.409952 155.649998)
+        (xy 206.290035 155.65)
         (xy 206.29 135)
         (xy 215.41 134.999998)
@@
     (polygon
       (pts
-        (xy 144.29 145.24)
-        (xy 144.29 155.24)
-        (xy 135.17 155.24)
-        (xy 135.17 145.24)
+        (xy 144.29 145.65)
+        (xy 144.29 155.65)
+        (xy 135.17 155.65)
+        (xy 135.17 145.65)
         (xy 137.16 138.43)
         (xy 142.24 138.43)
@@
     (polygon
       (pts
-        (xy 73.17 155.24)
-        (xy 64.05 155.24)
+        (xy 73.17 155.65)
+        (xy 64.05 155.65)
         (xy 64.05 135)
         (xy 73.17 135)
